Commit message: Update my_robot.xacro

File: 2-go-chase-robot/src/my_robot/urdf/my_robot.xacro (robot description, xacro)
@@ -1,176 +1,186 @@
 <?xml version='1.0'?>
 <robot name="my_robot" xmlns:xacro="http://www.ros.org/wiki/xacro">
-    <xacro:include filename="$(find my_robot)/urdf/my_robot.gazebo" />
-    <link name="robot_footprint"></link>
-    <joint name="robot_footprint_joint" type="fixed">
-        <origin xyz="0 0 0" rpy="0 0 0" />
-        <parent link="robot_footprint" />
-        <child link="chassis" />
-    </joint>
-    <link name='chassis'>
-        <pose>0 0 0.1 0 0 0</pose>
-        <inertial>
-            <mass value="15.0" />
-            <origin xyz="0.0 0 0" rpy=" 0 0 0" />
-            <inertia ixx="0.1" ixy="0" ixz="0" iyy="0.1" iyz="0" izz="0.1" />
-        </inertial>
-        <collision name='collision'>
-            <origin xyz="0 0 0" rpy=" 0 0 0" />
-            <geometry>
-                <box size=".4 .2 .1" />
-            </geometry>
-        </collision>
-        <visual name='chassis_visual'>
-            <origin xyz="0 0 0" rpy=" 0 0 0" />
-            <geometry>
-                <box size=".4 .2 .1" />
-            </geometry>
-        </visual>
-        <collision name='back_caster_collision'>
-            <origin xyz="-0.15 0 -0.05" rpy=" 0 0 0" />
-            <geometry>
-                <sphere radius="0.0499" />
-            </geometry>
-        </collision>
-        <visual name='back_caster_visual'>
-            <origin xyz="-0.15 0 -0.05" rpy=" 0 0 0" />
-            <geometry>
-                <sphere radius="0.05" />
-            </geometry>
-        </visual>
-        <collision name='front_caster_collision'>
-            <origin xyz="0.15 0 -0.05" rpy=" 0 0 0" />
-            <geometry>
-                <sphere radius="0.0499" />
-            </geometry>
-        </collision>
-        <visual name='front_caster_visual'>
-            <origin xyz="0.15 0 -0.05" rpy=" 0 0 0" />
-            <geometry>
-                <sphere radius="0.05" />
-            </geometry>
-        </visual>
-    </link>
-    <!-- my enhancements
-   -->
-    <link name="left_wheel">
-        <inertial>
-            <mass value="5.0" />
-            <origin xyz="0.0 0 0" rpy=" 0 1.5707 1.5707" />
-            <inertia ixx="0.1" ixy="0" ixz="0" iyy="0.1" iyz="0" izz="0.1" />
-        </inertial>
-        <collision name='left_wheel_collision'>
-            <origin xyz="0 0 0" rpy=" 0 1.5707 1.5707" />
-            <geometry>
-                <cylinder length="0.05" radius="0.1" />
-            </geometry>
-        </collision>
-        <visual name='left_wheel_visual'>
-            <origin xyz="0 0 0" rpy=" 0 1.5705 1.5707" />
-            <geometry>
-                <cylinder length="0.05" radius="0.1" />
-            </geometry>
-        </visual>
-    </link>
-    <joint type="continuous" name="left_wheel_hinge">
-        <origin xyz="0 0.15 0" rpy="0 0 0" />
-        <child link="left_wheel" />
-        <parent link="chassis" />
-        <axis xyz="0 1 0" rpy="0 0 0" />
-        <limit effort="10000" velocity="1000" />
-        <dynamics damping="1.0" friction="1.0" />
-    </joint>
-    <link name="right_wheel">
-        <inertial>
-            <mass value="5.0" />
-            <origin xyz="0 0 0" rpy=" 0 1.5707 1.5707" />
-            <inertia ixx="0.1" ixy="0" ixz="0" iyy="0.1" iyz="0" izz="0.1" />
-        </inertial>
-        <collision name='right_wheel_collision'>
-            <origin xyz="0 0 0" rpy=" 0 1.5707 1.5707" />
-            <geometry>
-                <cylinder length="0.05" radius="0.1" />
-            </geometry>
-        </collision>
-        <visual name='right_wheel_visual'>
-            <origin xyz="0 0 0" rpy=" 0 1.5705 1.5707" />
-            <geometry>
-                <cylinder length="0.05" radius="0.1" />
-            </geometry>
-        </visual>
-    </link>
-    <joint type="continuous" name="right_wheel_hinge">
-        <origin xyz="0 -0.15 0" rpy="0 0 0" />
-        <child link="right_wheel" />
-        <parent link="chassis" />
-        <axis xyz="0 1 0" rpy="0 0 0" />
-        <limit effort="10000" velocity="1000" />
-        <dynamics damping="1.0" friction="1.0" />
-    </joint>
-    <!-- Camera  -->
-    <link name="camera">
-        <inertial>
-            <mass value="0.1" />
-            <origin xyz="0 0 0" rpy=" 0 0 0" />
-            <inertia ixx="1e-6" ixy="0" ixz="0" iyy="1e-6" iyz="0" izz="1e-6" />
-        </inertial>
-        <collision name='camera_collision'>
-            <origin xyz="0 0 0" rpy=" 0 0 0" />
-            <geometry>
-                <box size="0.05 0.05 0.05" />
-            </geometry>
-        </collision>
-        <visual name='camera_visual'>
-            <origin xyz="0 0 0" rpy=" 0 0 0" />
-            <geometry>
-                <box size="0.05 0.05 0.05" />
-            </geometry>
-        </visual>
-    </link>
-    <!-- Camera Joint -->
-    <joint type="fixed" name="camera_joint">
-        <origin xyz="0.2 0 0" rpy="0 0 0" />
-        <child link="camera" />
-        <parent link="chassis" />
-        <axis xyz="0 1 0" rpy="0 0 0" />
-    </joint>
-    <!-- Lidar -->
-    <link name="hokuyo">
-        <inertial>
-            <mass value="1e-5" />
-            <origin xyz="0 0 0" rpy=" 0 0 0" />
-            <inertia ixx="1e-6" ixy="0" ixz="0" iyy="1e-6" iyz="0" izz="1e-6" />
-        </inertial>
-        <collision name='hokuyo_collision'>
-            <origin xyz="0 0 0" rpy=" 0 0 0" />
-            <geometry>
-                <box size="0.1 0.1 0.1" />
-            </geometry>
-        </collision>
-        <visual name='hokuyo_visual'>
-            <origin xyz="0 0 0" rpy=" 0 0 0" />
-            <geometry>
-                <mesh filename="package://my_robot/meshes/hokuyo.dae" />
-            </geometry>
-        </visual>
-    </link>
-    <joint type="fixed" name="hokuyo_joint">
-        <origin xyz="0.15 0 0.1" rpy="0 0 0" />
-        <child link="hokuyo" />
-        <parent link="chassis" />
-        <axis xyz="0 1 0" rpy="0 0 0" />
-    </joint>
-    <!-- Color  -->
-    <gazebo reference="chassis">
-        <material>Gazebo/Red</material>
-    </gazebo>
-    <gazebo reference="camera">
-        <material>Gazebo/Blue</material>
-    </gazebo>
-    <gazebo reference="left_wheel">
-        <material>Gazebo/Black</material>
-    </gazebo>
-    <gazebo reference="right_wheel">
-        <material>Gazebo/Black</material>
-    </gazebo>
-</robot>
+  <xacro:include filename="$(find my_robot)/urdf/my_robot.gazebo" />
+  <link name="robot_footprint"></link>
+  <joint name="robot_footprint_joint" type="fixed">
+    <origin xyz="0 0 0" rpy="0 0 0" />
+    <parent link="robot_footprint"/>
+    <child link="chassis" />
+  </joint>
+  <link name='chassis'>
+    <pose>0 0 0.1 0 0 0</pose>
+    <inertial>
+      <mass value="15.0"/>
+      <origin xyz="0.0 0 0" rpy=" 0 0 0"/>
+      <inertia
+              ixx="0.1" ixy="0" ixz="0"
+              iyy="0.1" iyz="0"
+              izz="0.1"
+      />
+    </inertial>
+    <collision name='collision'>
+      <origin xyz="0 0 0" rpy=" 0 0 0"/>
+      <geometry>
+        <box size=".4 .2 .1"/>
+      </geometry>
+    </collision>
+    <visual name='chassis_visual'>
+      <origin xyz="0 0 0" rpy=" 0 0 0"/>
+      <geometry>
+        <box size=".4 .2 .1"/>
+      </geometry>
+    </visual>
+    <collision name='back_caster_collision'>
+      <origin xyz="-0.15 0 -0.05" rpy=" 0 0 0"/>
+      <geometry>
+        <sphere radius="0.0499"/>
+      </geometry>
+    </collision>
+    <visual name='back_caster_visual'>
+      <origin xyz="-0.15 0 -0.05" rpy=" 0 0 0"/>
+      <geometry>
+        <sphere radius="0.05"/>
+      </geometry>
+    </visual>
+    <collision name='front_caster_collision'>
+      <origin xyz="0.15 0 -0.05" rpy=" 0 0 0"/>
+      <geometry>
+        <sphere radius="0.0499"/>
+      </geometry>
+    </collision>
+    <visual name='front_caster_visual'>
+      <origin xyz="0.15 0 -0.05" rpy=" 0 0 0"/>
+      <geometry>
+        <sphere radius="0.05"/>
+      </geometry>
+    </visual>
+  </link>
+  <!-- Add two wheels -->
+  <link name="left_wheel">
+    <inertial>
+      <origin xyz="0 0 0" rpy="0 1.5707 1.5707"/>
+      <mass value="5"/>
+      <inertia
+              ixx="0.1" ixy="0" ixz="0"
+              iyy="0.1" iyz="0" izz="0.1"
+      />
+    </inertial>
+    <collision>
+      <origin xyz="0 0 0" rpy="0 1.5707 1.5707"/>
+      <geometry>
+        <cylinder radius="0.1" length="0.05"/>
+      </geometry>
+    </collision>
+    <visual>
+      <origin xyz="0 0 0" rpy="0 1.5707 1.5707"/>
+      <geometry>
+        <cylinder radius="0.1" length="0.05"/>
+      </geometry>
+    </visual>
+  </link>
+  <link name="right_wheel">
+    <inertial>
+      <origin xyz="0 0 0" rpy="0 1.5707 1.5707"/>
+      <mass value="5"/>
+      <inertia
+              ixx="0.1" ixy="0" ixz="0"
+              iyy="0.1" iyz="0" izz="0.1"
+      />
+    </inertial>
+    <collision>
+      <origin xyz="0 0 0" rpy="0 1.5707 1.5707"/>
+      <geometry>
+        <cylinder radius="0.1" length="0.05"/>
+      </geometry>
+    </collision>
+    <visual>
+      <origin xyz="0 0 0" rpy="0 1.5707 1.5707"/>
+      <geometry>
+        <cylinder radius="0.1" length="0.05"/>
+      </geometry>
+    </visual>
+  </link>
+  <joint name="left_wheel_hinge" type="continuous">
+    <origin xyz="0 0.125 0" rpy="0 0 0"/>
+    <child link="left_wheel"/>
+    <parent link="chassis"/>
+    <axis xyz="0 1 0" rpy="0 0 0"/>
+    <limit effort="10000" velocity="1000"/>
+    <dynamics damping="1.0" friction="1.0"/>
+  </joint>
+  <joint name="right_wheel_hinge" type="continuous">
+    <origin xyz="0 -0.125 0" rpy="0 0 0"/>
+    <child link="right_wheel"/>
+    <parent link="chassis"/>
+    <axis xyz="0 1 0" rpy="0 0 0"/>
+    <limit effort="10000" velocity="1000"/>
+    <dynamics damping="1.0" friction="1.0"/>
+  </joint>
+  <!-- Add camera -->
+  <link name="camera">
+    <origin xyz="0 0 0" rpy="0 0 0" />
+    <inertial>
+      <mass value="0.1"/>
+      <inertia
+              ixx="1e-6" ixy="0" ixz="0"
+              iyy="1e-6" iyz="0" izz="1e-6"
+      />
+    </inertial>
+    <collision>
+      <geometry>
+        <box size="0.05 0.05 0.05"/>
+      </geometry>
+    </collision>
+    <visual>
+      <geometry>
+        <box size="0.05 0.05 0.05"/>
+      </geometry>
+    </visual>
+  </link>
+  <joint name="camera_joint" type="fixed">
+    <axis xyz="0 1 0"/>
+    <origin xyz="0.2 0 0" rpy="0 0 0" />
+    <parent link="chassis"/>
+    <child link="camera" />
+  </joint>
+  <!-- Add Lidar -->
+  <link name="hokuyo">
+    <origin xyz="0 0 0" rpy="0 0 0" />
+    <inertial>
+      <mass value="1e-5"/>
+      <inertia
+              ixx="1e-6" ixy="0" ixz="0"
+              iyy="1e-6" iyz="0" izz="1e-6"
+      />
+    </inertial>
+    <collision>
+      <geometry>
+        <box size=".1 .1 .1"/>
+      </geometry>
+    </collision>
+    <visual>
+      <geometry>
+        <mesh filename="package://my_robot/meshes/hokuyo.dae"/>
+      </geometry>
+    </visual>
+  </link>
+  <joint name="hokuyo_joint" type="fixed">
+    <axis xyz="0 1 0"/>
+    <origin xyz="0.15 0 0.1" rpy="0 0 0" />
+    <parent link="chassis"/>
+    <child link="hokuyo" />
+  </joint>
+  <!-- Color the components -->
+  <gazebo reference="chassis">
+    <material>Gazebo/Orange</material>
+  </gazebo>
+  <gazebo reference="left_wheel">
+    <material>Gazebo/Green</material>
+  </gazebo>
+  <gazebo reference="right_wheel">
+    <material>Gazebo/Green</material>
+  </gazebo>
+  <gazebo reference="camera">
+    <material>Gazebo/Red</material>
+  </gazebo>
+  </robot>

Commit message: fix: assaignment dimenstions

File: 2-go-chase-robot/src/my_robot/urdf/my_robot.xacro (robot description, xacro)
@@ -18,5 +18,5 @@
             <origin xyz="0 0 0" rpy=" 0 0 0" />
             <geometry>
-                <box size=".4 .2 .1" />
+                <box size=".412 .206 .103" /> <!-- BEGIN: Adjusted chassis dimensions -->
             </geometry>
         </collision>
@@ -24,5 +24,5 @@
             <origin xyz="0 0 0" rpy=" 0 0 0" />
             <geometry>
-                <box size=".4 .2 .1" />
+                <box size=".412 .206 .103" /> <!-- BEGIN: Adjusted chassis dimensions -->
             </geometry>
         </visual>
@@ -63,5 +63,5 @@
             <origin xyz="0 0 0" rpy=" 0 1.5707 1.5707" />
             <geometry>
-                <cylinder length="0.05" radius="0.1" />
+                <cylinder length="0.05" radius="0.103" /> <!-- BEGIN: Adjusted wheel radius -->
             </geometry>
         </collision>
@@ -69,5 +69,5 @@
             <origin xyz="0 0 0" rpy=" 0 1.5705 1.5707" />
             <geometry>
-                <cylinder length="0.05" radius="0.1" />
+                <cylinder length="0.05" radius="0.103" /> <!-- BEGIN: Adjusted wheel radius -->
             </geometry>
         </visual>
@@ -90,5 +90,5 @@
             <origin xyz="0 0 0" rpy=" 0 1.5707 1.5707" />
             <geometry>
-                <cylinder length="0.05" radius="0.1" />
+                <cylinder length="0.05" radius="0.103" /> <!-- BEGIN: Adjusted wheel radius -->
             </geometry>
         </collision>
@@ -96,5 +96,5 @@
             <origin xyz="0 0 0" rpy=" 0 1.5705 1.5707" />
             <geometry>
-                <cylinder length="0.05" radius="0.1" />
+                <cylinder length="0.05" radius="0.103" /> <!-- BEGIN: Adjusted wheel radius -->
             </geometry>
         </visual>
